Commit message: Move body assets out of the robot with instance-based naming

File: assets/common/assembly.xacro (robot description, xacro)
@@ -98,6 +98,5 @@
       <xacro:property name="parent_reference_emitted" value="${parent_ref.get('emit', False)}" lazy_eval="false" />
       <xacro:if value="${parent_reference_emitted}">
-        <xacro:property name="reference_prefix" value="${parent_desc['reference_prefix']}" lazy_eval="false" />
-        <xacro:property name="resolved_connected_to" value="${reference_prefix + parent_ref_name}" lazy_eval="false" />
+        <xacro:property name="resolved_connected_to" value="${parent_desc['prefix'] + parent_ref_name}" lazy_eval="false" />
         <xacro:property name="resolved_mount_origin" value="${connection_origin}" lazy_eval="false" />
       </xacro:if>

File: assets/common/components.xacro (robot description, xacro)
@@ -41,7 +41,7 @@
     <xacro:property name="component_visuals" value="${xacro.load_yaml(component_cfg_root + '/link/visuals.yaml')}" lazy_eval="false" />
     <xacro:property name="component_collisions" value="${xacro.load_yaml(component_cfg_root + '/link/collisions.yaml')}" lazy_eval="false" />
-    <xacro:property name="component_link_name_map" value="${dict([(component_topology['links'][0], component_cfg['link_name'])]) if component_type == 'body' else empty_dict}" lazy_eval="false" />
-    <xacro:property name="component_root_link_actual" value="${component_cfg['link_name'] if component_type == 'body' else (component_prefix + component_topology['links'][0])}" lazy_eval="false" />
-    <xacro:property name="component_default_mount_parent" value="${component_cfg['link_name'] if component_type == 'body' else (component_prefix + component_topology['links'][-1])}" lazy_eval="false" />
+    <xacro:property name="component_link_name_map" value="${empty_dict}" lazy_eval="false" />
+    <xacro:property name="component_root_link_actual" value="${component_prefix + component_topology['links'][0]}" lazy_eval="false" />
+    <xacro:property name="component_default_mount_parent" value="${component_prefix + (component_topology['links'][0] if component_type == 'body' else component_topology['links'][-1])}" lazy_eval="false" />
     <xacro:property name="component_collapse_empty_end" value="${component_type == 'arm' and options.get('collapse_empty_end', False) and len([j for j in component_topology['joints'] if component_topology['joints'][j]['parent'] == component_topology['links'][-1]]) == 0}" lazy_eval="false" />
     <xacro:property
@@ -67,6 +67,5 @@
                    default_mount_parent=component_default_mount_parent,
                    collapse_empty_end=component_collapse_empty_end,
-                   supports_frame_shift=True,
-                   reference_prefix=(component_root_link_actual + '_' if component_type == 'body' else component_prefix))}"
+                   supports_frame_shift=True)}"
       scope="parent"
       lazy_eval="false" />
@@ -116,6 +115,5 @@
     <xacro:openarm_emit_reference_frames
       reference_points="${component_desc['reference_points']}"
-      prefix="${component_desc['reference_prefix']}"
-      link_prefix="${component_desc['prefix']}"
+      prefix="${component_desc['prefix']}"
       link_name_map="${component_desc['link_name_map']}"
       base_link_name="${component_desc['topology']['links'][0]}"

File: assets/common/reference_frames.xacro (robot description, xacro)
@@ -28,5 +28,5 @@
   </xacro:macro>
   <xacro:macro name="openarm_emit_reference_frames"
-    params="reference_points prefix link_prefix link_name_map:=${dict()} base_link_name:='' reflect_x:=1 reflect_y:=1 reflect_z:=1 reflect_include_reference_points:=^ frame_shift:=none force_emit_reference:='' index:=0">
+    params="reference_points prefix link_name_map:=${dict()} base_link_name:='' reflect_x:=1 reflect_y:=1 reflect_z:=1 reflect_include_reference_points:=^ frame_shift:=none force_emit_reference:='' index:=0">
     <xacro:property name="reference_names" value="${list(reference_points.keys())}" lazy_eval="false" />
     <xacro:if value="${index &lt; len(reference_names)}">
@@ -38,5 +38,5 @@
         <xacro:openarm_emit_reference_link
           link_name="${prefix + reference_name}"
-          parent_link="${link_name_map[reference_parent] if reference_parent in link_name_map else link_prefix + reference_parent}"
+          parent_link="${link_name_map[reference_parent] if reference_parent in link_name_map else prefix + reference_parent}"
           origin="${reference['origin']}"
           reflect_x="${reflect_x if reference_reflects else 1}"
@@ -46,5 +46,5 @@
       </xacro:if>
       <xacro:openarm_emit_reference_frames
-        reference_points="${reference_points}" prefix="${prefix}" link_prefix="${link_prefix}"
+        reference_points="${reference_points}" prefix="${prefix}"
         link_name_map="${link_name_map}" base_link_name="${base_link_name}"
         reflect_x="${reflect_x}" reflect_y="${reflect_y}" reflect_z="${reflect_z}"

File: assets/common/validation.xacro (robot description, xacro)
@@ -75,6 +75,6 @@
       </xacro:if>
       <xacro:if value="${component_type == 'body'}">
-        <xacro:openarm_require condition="${component_config == None and 'link_name' in component_cfg}"
-          message="${'Body `%s` requires config: null and link_name.' % component_name}" />
+        <xacro:openarm_require condition="${component_config == None}"
+          message="${'Body `%s` requires config: null.' % component_name}" />
       </xacro:if>
       <xacro:openarm_require

File: assets/end_effector/pinch_gripper/urdf/pinch_gripper_macro.xacro (robot description, xacro)
@@ -157,5 +157,5 @@
       reference_points="${ee_reference_points}"
       force_emit_reference="${grasp_reference_point if emit_grasp_frame else ''}"
-      prefix="${prefix}" link_prefix="${prefix}"
+      prefix="${prefix}"
       base_link_name="${base_link_name}"
       reflect_x="${reflect_x if component_reflects else 1}"

File: assets/robot/openarm_v2.0/urdf/example/v2.urdf (robot description, URDF)
Before this commit: robot openarm_v20, 24 links, 23 joints
Links:
- link openarm_body_link0: geometry collision mesh filename=package://openarm_description/assets/body/v2.0/meshes/colli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 scale=0.001 0.001 0.001; visual mesh filename=package://openarm_description/assets/body/v2.0/meshes/visua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 scale=1.0 1.0 1.0

File: assets/sensor/zed/urdf/component.xacro (robot description, xacro)
@@ -46,5 +46,4 @@
                    collapse_empty_end=False,
                    supports_frame_shift=False,
-                   reference_prefix=component_prefix,
                    config_root=config_root)}"
       scope="parent"
