Commit message: Generate arm and gripper joints from topology

File: assets/common/assembly.xacro (robot description, xacro)
@@ -70,5 +70,5 @@
       <xacro:property name="parent_ref_canonical_link" value="${parent_ref['parent']}" lazy_eval="false" />
       <xacro:property name="resolved_connected_to"
-        value="${parent_desc['link_name_map'][parent_ref_canonical_link] if parent_ref_canonical_link in parent_desc['link_name_map'] else parent_desc['link_prefix'] + parent_ref_canonical_link}" lazy_eval="false" />
+        value="${parent_desc['link_name_map'][parent_ref_canonical_link] if parent_ref_canonical_link in parent_desc['link_name_map'] else parent_desc['prefix'] + parent_ref_canonical_link}" lazy_eval="false" />
       <xacro:property name="reference_origin" value="${parent_ref['origin']}" lazy_eval="false" />
       <xacro:if value="${parent_ref_canonical_link == parent_desc['topology']['links'][0] and parent_desc.get('base_frame_shift', 'none') != 'none'}">
@@ -94,5 +94,5 @@
     <xacro:if value="${has_parent_reference_key and not has_parent_override and collapse_internal_empty_links and parent_terminal_link_empty and parent_ref_canonical_link == parent_desc['topology']['links'][-1]}">
       <xacro:property name="skip_mount_joint" value="${True}" lazy_eval="false" />
-      <xacro:openarm_reflect_pose origin="${reference_mount_origin}" reflect_x="${reflect_x}" reflect_y="${reflect_y}" reflect_z="${reflect_z}" out_name="base_frame_shift" />
+  <xacro:openarm_reflect_pose origin="${reference_mount_origin}" reflect_x="${reflect_x}" reflect_y="${reflect_y}" reflect_z="${reflect_z}" out_name="base_frame_shift" />
     </xacro:if>
     <!-- A parent can expose at most one child that consumes its terminal empty link. -->

File: assets/common/validation.xacro (robot description, xacro)
@@ -113,3 +113,25 @@
       robot_preset="${robot_preset}" />
   </xacro:macro>
+  <xacro:macro name="openarm_validate_link_ancestry" params="name topology component depth:=0">
+    <xacro:if value="${name != topology['links'][0]}">
+      <xacro:openarm_require condition="${depth &lt; len(topology['links'])}" message="${'Component `%s` has a cycle at link `%s`.' % (component, name)}" />
+      <xacro:property name="incoming" value="${[j for j in topology['joints'] if topology['joints'][j]['child'] == name]}" lazy_eval="false" />
+      <xacro:openarm_require condition="${len(incoming) == 1}" message="${'Link `%s` in `%s` must have one parent joint.' % (name, component)}" />
+      <xacro:openarm_validate_link_ancestry name="${topology['joints'][incoming[0]]['parent']}" topology="${topology}" component="${component}" depth="${depth + 1}" />
+    </xacro:if>
+  </xacro:macro>
+  <xacro:macro name="openarm_validate_topology" params="topology component index:=0">
+    <xacro:property name="links" value="${topology['links']}" lazy_eval="false" />
+    <xacro:property name="joints" value="${topology['joints']}" lazy_eval="false" />
+    <xacro:if value="${index == 0}">
+      <xacro:openarm_require condition="${len(links) > 0 and len([link for link in links if links.count(link) != 1]) == 0}" message="${'Component `%s` must have nonempty, unique links.' % component}" />
+      <xacro:openarm_require condition="${len([j for j in joints if joints[j]['parent'] not in links or joints[j]['child'] not in links]) == 0}" message="${'Component `%s` has a joint referencing an unknown link.' % component}" />
+      <xacro:openarm_require condition="${len([j for j in joints if joints[j]['child'] == links[0]]) == 0}" message="${'Root link of `%s` cannot have an internal parent joint.' % component}" />
+      <xacro:openarm_require condition="${len([j for j in joints if joints[j]['type'] not in ['fixed', 'revolute', 'continuous', 'prismatic']]) == 0}" message="${'Component `%s` has an unsupported joint type.' % component}" />
+    </xacro:if>
+    <xacro:if value="${index &lt; len(links)}">
+      <xacro:openarm_validate_link_ancestry name="${links[index]}" topology="${topology}" component="${component}" />
+      <xacro:openarm_validate_topology topology="${topology}" component="${component}" index="${index + 1}" />
+    </xacro:if>
+  </xacro:macro>
 </robot>

File: assets/component_loader.xacro (robot description, xacro)
@@ -16,7 +16,7 @@
   <xacro:include filename="$(find openarm_description)/assets/common/reference_frames.xacro" />
   <xacro:include filename="$(find openarm_description)/assets/common/validation.xacro" />
-  <xacro:include filename="$(find openarm_description)/assets/robot/openarm_v2.0/urdf/utils/openarm_v20_arm.xacro" />
+  <xacro:include filename="$(find openarm_description)/assets/common/kinematic_chain.xacro" />
   <xacro:include filename="$(find openarm_description)/assets/end_effector/pinch_gripper/urdf/pinch_gripper_macro.xacro" />
-  <xacro:include filename="$(find openarm_description)/assets/robot/openarm_v2.0/urdf/utils/openarm_v20_sensor.xacro" />
+  <xacro:include filename="$(find openarm_description)/assets/sensor/zed/urdf_wrapper/openarm_zed_wrapper.xacro" />
   <xacro:macro name="openarm_load_component_descriptor"
     params="component_name component_cfg config_root out_name">
@@ -31,4 +31,8 @@
         message="${'Invalid robot preset: robot component `%s` uses unsupported product `%s`.' % (component_name, component_cfg['product'])}" />
     </xacro:if>
+    <xacro:if value="${source_type == 'end_effector'}">
+      <xacro:openarm_require condition="${component_cfg['product'] == 'pinch_gripper'}"
+        message="${'Unsupported end effector `%s`.' % component_cfg['product']}" />
+    </xacro:if>
     <xacro:if value="${source_type == 'sensor'}">
       <xacro:openarm_require
@@ -50,5 +54,4 @@
                      config=component_config,
                      prefix=component_prefix,
-                     link_prefix=component_prefix,
                      root_link_actual=sensor_root_link,
                      topology=dict(links=[sensor_root_link], joints=dict()),
@@ -79,6 +82,6 @@
           lazy_eval="false" />
       </xacro:if>
-      <xacro:property name="component_link_prefix" value="${component_prefix + ('ee_' if component_type == 'end_effector' else '')}" lazy_eval="false" />
       <xacro:property name="component_topology" value="${xacro.load_yaml(component_cfg_root + '/struct/topology.yaml')}" lazy_eval="false" />
+      <xacro:openarm_validate_topology topology="${component_topology}" component="${component_name}" />
       <xacro:property name="component_reference_points" value="${xacro.load_yaml(component_cfg_root + '/struct/reference_points.yaml')}" lazy_eval="false" />
       <xacro:property name="component_joint_origins" value="${xacro.load_yaml(component_cfg_root + '/joint/joint_origins.yaml') if component_type != 'body' else empty_dict}" lazy_eval="false" />
@@ -90,6 +93,6 @@
       <xacro:property name="component_collisions" value="${xacro.load_yaml(component_cfg_root + '/link/collisions.yaml')}" lazy_eval="false" />
       <xacro:property name="component_link_name_map" value="${dict(body_link0=component_cfg['link_name']) if component_type == 'body' else empty_dict}" lazy_eval="false" />
-      <xacro:property name="component_root_link_actual" value="${component_cfg['link_name'] if component_type == 'body' else (component_link_prefix + component_topology['links'][0])}" lazy_eval="false" />
-      <xacro:property name="component_default_mount_parent" value="${component_cfg['link_name'] if component_type == 'body' else (component_link_prefix + component_topology['links'][-1])}" lazy_eval="false" />
+      <xacro:property name="component_root_link_actual" value="${component_cfg['link_name'] if component_type == 'body' else (component_prefix + component_topology['links'][0])}" lazy_eval="false" />
+      <xacro:property name="component_default_mount_parent" value="${component_cfg['link_name'] if component_type == 'body' else (component_prefix + component_topology['links'][-1])}" lazy_eval="false" />
       <xacro:property name="component_supports_tip_collapse" value="${component_type == 'arm'}" lazy_eval="false" />
       <xacro:property
@@ -102,5 +105,4 @@
                      config_root=component_cfg_root,
                      prefix=component_prefix,
-                     link_prefix=component_link_prefix,
                      root_link_actual=component_root_link_actual,
                      topology=component_topology,
@@ -140,5 +142,5 @@
     </xacro:if>
     <xacro:if value="${component_type == 'arm'}">
-      <xacro:openarm_v20_arm
+      <xacro:openarm_emit_kinematic_component
         prefix="${component_desc['prefix']}"
         connected_to="${component_runtime['resolved_connected_to']}"
@@ -148,4 +150,5 @@
         joint_axes="${component_desc['joint_axes']}"
         joint_limits="${component_desc['joint_limits']}"
+        joint_mimics="${component_desc['joint_mimics']}"
         inertials="${component_desc['inertials']}"
         visuals="${component_desc['visuals']}"
@@ -154,5 +157,4 @@
         reflect_y="${component_runtime['reflect_y']}"
         reflect_z="${component_runtime['reflect_z']}"
-        component_reflects="${component_runtime['component_reflects']}"
         reflect_include_links="${component_runtime['reflect_include_links']}"
         reflect_include_joints="${component_runtime['reflect_include_joints']}"
@@ -163,5 +165,5 @@
         base_frame_shift="${component_runtime['base_frame_shift']}" />
     </xacro:if>
-    <xacro:if value="${component_type == 'end_effector'}">
+    <xacro:if value="${component_type == 'end_effector' and component_desc['product'] == 'pinch_gripper'}">
       <xacro:openarm_pinch_gripper
         prefix="${component_desc['prefix']}"
@@ -190,6 +192,5 @@
     </xacro:if>
     <xacro:if value="${component_type == 'sensor'}">
-      <xacro:openarm_v20_sensor
-        product="${component_desc['product']}"
+      <xacro:openarm_zed_wrapper
         config="${component_desc['config']}"
         connected_to="${component_runtime['resolved_connected_to']}"
@@ -197,9 +198,9 @@
         prefix="${component_desc['prefix']}" />
     </xacro:if>
-    <xacro:unless value="${component_type == 'end_effector'}">
+    <xacro:unless value="${component_type == 'end_effector' and component_desc['product'] == 'pinch_gripper'}">
       <xacro:openarm_emit_reference_frames
         reference_points="${component_desc['reference_points']}"
         prefix="${component_desc['root_link_actual'] + '_' if component_type == 'body' else component_desc['prefix']}"
-        link_prefix="${component_desc['link_prefix']}"
+        link_prefix="${component_desc['prefix']}"
         link_name_map="${component_desc['link_name_map']}"
         base_link_name="${component_desc['topology']['links'][0]}"

File: assets/end_effector/pinch_gripper/urdf/pinch_gripper_macro.xacro (robot description, xacro)
@@ -15,10 +15,9 @@
   <xacro:include filename="$(find openarm_description)/assets/common/links.xacro" />
   <xacro:include filename="$(find openarm_description)/assets/common/reference_frames.xacro" />
-  <!-- Current EE implementation targets the two-finger gripper topology. -->
   <xacro:include filename="$(find openarm_description)/assets/common/validation.xacro" />
   <xacro:macro name="openarm_pinch_gripper"
     params="prefix connected_to mount_origin:=none topology joint_origins joint_axes joint_limits joint_mimics inertials visuals collisions reflect_x:=1 reflect_y:=1 reflect_z:=1 component_reflects:=false reflect_include_links:=^ reflect_include_joints:=^ reflect_include_reference_points:=^ limit_override_joints:=^ ee_reference_points:=^ emit_grasp_frame:=false grasp_reference_point:=grasp_frame skip_mount_joint:=false base_frame_shift:=none">
     <xacro:property name="base_link_name" value="${topology['links'][0]}" />
-    <xacro:property name="base_link_full_name" value="${prefix}ee_${base_link_name}" />
+    <xacro:property name="base_link_full_name" value="${prefix}${base_link_name}" />
     <xacro:property name="resolved_mount_origin" value="${mount_origin if mount_origin != 'none' else dict(x=0.0, y=0.0, z=0.0, roll=0.0, pitch=0.0, yaw=0.0)}" lazy_eval="false" />
     <xacro:property name="resolved_base_frame_shift" value="${base_frame_shift if base_frame_shift != 'none' else dict(x=0.0, y=0.0, z=0.0, roll=0.0, pitch=0.0, yaw=0.0)}" lazy_eval="false" />
@@ -26,8 +25,8 @@
     <xacro:property name="base_link_reflects" value="${component_reflects and base_link_name in reflect_include_links}" lazy_eval="false" />
     <!-- Finger numbering stays semantic; handedness is handled by reflect_* and the joint config. -->
-    <xacro:property name="finger1_source" value="link1" />
-    <xacro:property name="finger2_source" value="link2" />
-    <xacro:property name="finger1_joint_source" value="joint1" />
-    <xacro:property name="finger2_joint_source" value="joint2" />
+    <xacro:property name="finger1_source" value="${topology['joints']['finger_joint1']['child']}" />
+    <xacro:property name="finger2_source" value="${topology['joints']['finger_joint2']['child']}" />
+    <xacro:property name="finger1_joint_source" value="finger_joint1" />
+    <xacro:property name="finger2_joint_source" value="finger_joint2" />
     <xacro:property name="finger1_link_reflects" value="${component_reflects and finger1_source in reflect_include_links}" lazy_eval="false" />
     <xacro:property name="finger2_link_reflects" value="${component_reflects and finger2_source in reflect_include_links}" lazy_eval="false" />
@@ -38,6 +37,6 @@
     <xacro:property name="finger1_mimic_target_source" value="${joint_mimics[finger1_joint_source]['joint'] if finger1_has_mimic else ''}" />
     <xacro:property name="finger2_mimic_target_source" value="${joint_mimics[finger2_joint_source]['joint'] if finger2_has_mimic else ''}" />
-    <xacro:property name="finger1_mimic_target_name" value="${prefix + ('finger_joint1' if finger1_mimic_target_source == finger1_joint_source else 'finger_joint2')}" />
-    <xacro:property name="finger2_mimic_target_name" value="${prefix + ('finger_joint1' if finger2_mimic_target_source == finger1_joint_source else 'finger_joint2')}" />
+    <xacro:property name="finger1_mimic_target_name" value="${prefix + finger1_mimic_target_source}" />
+    <xacro:property name="finger2_mimic_target_name" value="${prefix + finger2_mimic_target_source}" />
     <xacro:property name="finger1_mimic_override" value="${dict(joint=finger1_mimic_target_name, multiplier=joint_mimics[finger1_joint_source]['multiplier'], offset=joint_mimics[finger1_joint_source]['offset']) if finger1_has_mimic else 'none'}" />
     <xacro:property name="finger2_mimic_override" value="${dict(joint=finger2_mimic_target_name, multiplier=joint_mimics[finger2_joint_source]['multiplier'], offset=joint_mimics[finger2_joint_source]['offset']) if finger2_has_mimic else 'none'}" />
@@ -99,5 +98,5 @@
     </link>
     <xacro:openarm_emit_link
-      link_name="${prefix}ee_link1"
+      link_name="${prefix}${finger1_source}"
       source_name="${finger1_source}"
       inertials="${inertials}"
@@ -108,5 +107,5 @@
       reflect_z="${reflect_z if finger1_link_reflects else 1}" />
     <xacro:openarm_emit_link
-      link_name="${prefix}ee_link2"
+      link_name="${prefix}${finger2_source}"
       source_name="${finger2_source}"
       inertials="${inertials}"
@@ -148,19 +147,21 @@
     <xacro:property
       name="finger1_joint_limit_override"
-      value="${limit_override_joints[finger1_joint_source] if finger1_joint_source in limit_override_joints else (limit_override_joints['finger_joint1'] if 'finger_joint1' in limit_override_joints else 'none')}"
+      value="${limit_override_joints.get(finger1_joint_source, 'none')}"
       lazy_eval="false" />
     <xacro:property
       name="finger2_joint_limit_override"
-      value="${limit_override_joints[finger2_joint_source] if finger2_joint_source in limit_override_joints else (limit_override_joints['finger_joint2'] if 'finger_joint2' in limit_override_joints else 'none')}"
-      lazy_eval="false" />
+      value="${limit_override_joints.get(finger2_joint_source, 'none')}"
+      lazy_eval="false" />
+    <xacro:property name="finger1_joint_limit_base" value="${finger1_joint_limit_override if finger1_joint_limit_override != 'none' else finger1_joint_limit_cfg}" lazy_eval="false" />
     <xacro:property
       name="finger1_joint_limit_effective"
-      value="${finger1_joint_limit_override if finger1_joint_limit_override != 'none' else (dict(lower=(-finger1_joint_limit_cfg['upper']), upper=(-finger1_joint_limit_cfg['lower']), effort=finger1_joint_limit_cfg['effort'], velocity=finger1_joint_limit_cfg['velocity']) if finger1_limit_should_mirror else finger1_joint_limit_cfg)}"
-      lazy_eval="false" />
+      value="${dict(lower=(-finger1_joint_limit_base['upper']), upper=(-finger1_joint_limit_base['lower']), effort=finger1_joint_limit_base['effort'], velocity=finger1_joint_limit_base['velocity']) if finger1_limit_should_mirror else finger1_joint_limit_base}"
+      lazy_eval="false" />
+    <xacro:property name="finger2_joint_limit_base" value="${finger2_joint_limit_override if finger2_joint_limit_override != 'none' else finger2_joint_limit_cfg}" lazy_eval="false" />
     <xacro:property
       name="finger2_joint_limit_effective"
-      value="${finger2_joint_limit_override if finger2_joint_limit_override != 'none' else (dict(lower=(-finger2_joint_limit_cfg['upper']), upper=(-finger2_joint_limit_cfg['lower']), effort=finger2_joint_limit_cfg['effort'], velocity=finger2_joint_limit_cfg['velocity']) if finger2_limit_should_mirror else finger2_joint_limit_cfg)}"
-      lazy_eval="false" />
-    <joint name="${prefix}finger_joint1" type="revolute">
+      value="${dict(lower=(-finger2_joint_limit_base['upper']), upper=(-finger2_joint_limit_base['lower']), effort=finger2_joint_limit_base['effort'], velocity=finger2_joint_limit_base['velocity']) if finger2_limit_should_mirror else finger2_joint_limit_base}"
+      lazy_eval="false" />
+    <joint name="${prefix}${finger1_joint_source}" type="${topology['joints'][finger1_joint_source]['type']}">
       <xacro:if value="${use_base_frame_shift}">
         <xacro:openarm_emit_composed_origin first="${resolved_base_frame_shift}" second="${finger1_joint_origin_cfg}" reflect_x="${reflect_x if finger1_joint_reflects else 1}" reflect_y="${reflect_y if finger1_joint_reflects else 1}" reflect_z="${reflect_z if finger1_joint_reflects else 1}" />
@@ -169,6 +170,7 @@
         <xacro:openarm_emit_origin origin="${finger1_joint_origin_cfg}" reflect_x="${reflect_x if finger1_joint_reflects else 1}" reflect_y="${reflect_y if finger1_joint_reflects else 1}" reflect_z="${reflect_z if finger1_joint_reflects else 1}" />
       </xacro:unless>
-      <parent link="${base_link_full_name}" />
-      <child link="${prefix}ee_link1" />
+      <parent link="${prefix}${topology['joints'][finger1_joint_source]['parent']}" />
+      <child link="${prefix}${finger1_source}" />
+      <xacro:if value="${topology['joints'][finger1_joint_source]['type'] != 'fixed'}">
       <axis xyz="${finger1_joint_axis_reflect_sign * finger1_joint_axis_cfg.x} ${finger1_joint_axis_reflect_sign * finger1_joint_axis_cfg.y} ${finger1_joint_axis_reflect_sign * finger1_joint_axis_cfg.z}" />
       <xacro:openarm_emit_limit limit="${finger1_joint_limit_effective}" />
@@ -179,6 +181,7 @@
           offset="${finger1_mimic_override['offset']}" />
       </xacro:if>
+          </xacro:if>
     </joint>
-    <joint name="${prefix}finger_joint2" type="revolute">
+    <joint name="${prefix}${finger2_joint_source}" type="${topology['joints'][finger2_joint_source]['type']}">
       <xacro:if value="${use_base_frame_shift}">
         <xacro:openarm_emit_composed_origin first="${resolved_base_frame_shift}" second="${finger2_joint_origin_cfg}" reflect_x="${reflect_x if finger2_joint_reflects else 1}" reflect_y="${reflect_y if finger2_joint_reflects else 1}" reflect_z="${reflect_z if finger2_joint_reflects else 1}" />
@@ -187,6 +190,7 @@
         <xacro:openarm_emit_origin origin="${finger2_joint_origin_cfg}" reflect_x="${reflect_x if finger2_joint_reflects else 1}" reflect_y="${reflect_y if finger2_joint_reflects else 1}" reflect_z="${reflect_z if finger2_joint_reflects else 1}" />
       </xacro:unless>
-      <parent link="${base_link_full_name}" />
-      <child link="${prefix}ee_link2" />
+      <parent link="${prefix}${topology['joints'][finger2_joint_source]['parent']}" />
+      <child link="${prefix}${finger2_source}" />
+      <xacro:if value="${topology['joints'][finger2_joint_source]['type'] != 'fixed'}">
       <axis xyz="${finger2_joint_axis_reflect_sign * finger2_joint_axis_cfg.x} ${finger2_joint_axis_reflect_sign * finger2_joint_axis_cfg.y} ${finger2_joint_axis_reflect_sign * finger2_joint_axis_cfg.z}" />
       <xacro:openarm_emit_limit limit="${finger2_joint_limit_effective}" />
@@ -197,9 +201,10 @@
           offset="${finger2_mimic_override['offset']}" />
       </xacro:if>
+          </xacro:if>
     </joint>
     <xacro:openarm_emit_reference_frames
       reference_points="${ee_reference_points}"
       force_emit_reference="${grasp_reference_point if emit_grasp_frame else ''}"
-      prefix="${prefix}" link_prefix="${prefix + 'ee_'}"
+      prefix="${prefix}" link_prefix="${prefix}"
       base_link_name="${base_link_name}"
       reflect_x="${reflect_x if component_reflects else 1}"

File: assets/end_effector/pinch_gripper/urdf/pinch_gripper_standalone.urdf.xacro (robot description, xacro)
@@ -13,6 +13,4 @@
 -->
 <robot xmlns:xacro="http://www.ros.org/wiki/xacro" name="pinch_gripper">
-  <xacro:include filename="$(find openarm_description)/assets/common/links.xacro" />
-  <xacro:include filename="$(find openarm_description)/assets/common/reference_frames.xacro" />
   <xacro:include filename="$(find openarm_description)/assets/end_effector/pinch_gripper/urdf/pinch_gripper_macro.xacro" />
   <xacro:arg name="ee_config_dir" default="$(find openarm_description)/assets/end_effector/pinch_gripper/config" />

File: assets/robot/openarm_v2.0/urdf/openarm_v20.urdf.xacro (robot description, xacro)
@@ -35,5 +35,5 @@
   <xacro:property name="pinch_mimics_file" value="$(find openarm_description)/assets/end_effector/pinch_gripper/config/joint/joint_mimics.yaml" />
   <xacro:property name="pinch_mimics_dict" value="${xacro.load_yaml(pinch_mimics_file)}" />
-  <xacro:property name="pinch_finger_mimic_multiplier" value="${pinch_mimics_dict['joint2']['multiplier'] if 'joint2' in pinch_mimics_dict else 1.0}" />
+  <xacro:property name="pinch_finger_mimic_multiplier" value="${pinch_mimics_dict['finger_joint2']['multiplier'] if 'finger_joint2' in pinch_mimics_dict else 1.0}" />
   <xacro:openarm_bimanual_ros2_control
     arm_type="v20"
