Commit message: Compose component mounting transforms after reflection

File: assets/common/assembly.xacro (robot description, xacro)
@@ -29,4 +29,7 @@
     <xacro:property name="reflect_include_reference_points" value="${reflect_include_cfg['reference_points'] if 'reference_points' in reflect_include_cfg else list(component_desc['reference_points'].keys())}" lazy_eval="false" />
     <xacro:property name="limit_override_joints" value="${component_cfg['limit_override_joints'] if 'limit_override_joints' in component_cfg else dict()}" lazy_eval="false" />
+    <xacro:property name="origin_override_joints" value="${component_cfg.get('origin_override_joints', dict())}" lazy_eval="false" />
+    <xacro:openarm_require condition="${len([name for name in list(origin_override_joints) + list(limit_override_joints) if name not in component_desc['topology']['joints']]) == 0}"
+      message="${'Unknown joint override on component `%s`.' % component_name}" />
     <xacro:property name="connection" value="${component_cfg['connection'] if 'connection' in component_cfg else dict()}" lazy_eval="false" />
     <xacro:property name="parent_component_name" value="${connection['attach_to'] if 'attach_to' in connection else none_value}" lazy_eval="false" />
@@ -72,9 +75,9 @@
         value="${parent_desc['link_name_map'][parent_ref_canonical_link] if parent_ref_canonical_link in parent_desc['link_name_map'] else parent_desc['prefix'] + parent_ref_canonical_link}" lazy_eval="false" />
       <xacro:property name="reference_origin" value="${parent_ref['origin']}" lazy_eval="false" />
+      <xacro:if value="${parent_ref_should_reflect}">
+        <xacro:openarm_reflect_pose origin="${reference_origin}" reflect_x="${parent_reflect_cfg['x']}" reflect_y="${parent_reflect_cfg['y']}" reflect_z="${parent_reflect_cfg['z']}" out_name="reference_origin" />
+      </xacro:if>
       <xacro:if value="${parent_ref_canonical_link == parent_desc['topology']['links'][0] and parent_desc.get('base_frame_shift', 'none') != 'none'}">
         <xacro:openarm_compose_pose first="${parent_desc['base_frame_shift']}" second="${reference_origin}" out_name="reference_origin" />
-      </xacro:if>
-      <xacro:if value="${parent_ref_should_reflect}">
-        <xacro:openarm_reflect_pose origin="${reference_origin}" reflect_x="${parent_reflect_cfg['x']}" reflect_y="${parent_reflect_cfg['y']}" reflect_z="${parent_reflect_cfg['z']}" out_name="reference_origin" />
       </xacro:if>
       <xacro:openarm_compose_pose first="${reference_origin}" second="${connection_origin}" out_name="reference_mount_origin" />
@@ -94,5 +97,5 @@
     <xacro:if value="${has_parent_reference_key and not has_parent_override and collapse_internal_empty_links and parent_terminal_link_empty and parent_ref_canonical_link == parent_desc['topology']['links'][-1]}">
       <xacro:property name="skip_mount_joint" value="${True}" lazy_eval="false" />
-  <xacro:openarm_reflect_pose origin="${reference_mount_origin}" reflect_x="${reflect_x}" reflect_y="${reflect_y}" reflect_z="${reflect_z}" out_name="base_frame_shift" />
+      <xacro:property name="base_frame_shift" value="${reference_mount_origin}" lazy_eval="false" />
     </xacro:if>
     <!-- A parent can expose at most one child that consumes its terminal empty link. -->
@@ -136,4 +139,5 @@
                    reflect_include_reference_points=reflect_include_reference_points,
                    limit_override_joints=limit_override_joints,
+                   origin_override_joints=origin_override_joints,
                    resolved_connected_to=resolved_connected_to,
                    resolved_mount_origin=resolved_mount_origin,

File: assets/common/links.xacro (robot description, xacro)
@@ -27,8 +27,8 @@
           <xacro:property name="visual_cfg" value="${visual_override if visual_override != 'none' else visuals[source_name]}" lazy_eval="false" />
           <xacro:if value="${frame_shift != 'none'}">
-            <xacro:openarm_emit_composed_origin first="${frame_shift}" second="${visual_cfg.origin}" reflect_x="${reflect_x}" reflect_y="${reflect_y}" reflect_z="${reflect_z}" />
+            <xacro:openarm_emit_shifted_origin frame_shift="${frame_shift}" origin="${visual_cfg.origin}" reflect_x="${reflect_x}" reflect_y="${reflect_y}" reflect_z="${reflect_z}" reflect_rotation="${True}" />
           </xacro:if>
           <xacro:unless value="${frame_shift != 'none'}">
-            <xacro:openarm_emit_origin origin="${visual_cfg.origin}" reflect_x="${reflect_x}" reflect_y="${reflect_y}" reflect_z="${reflect_z}" />
+            <xacro:openarm_emit_origin origin="${visual_cfg.origin}" reflect_x="${reflect_x}" reflect_y="${reflect_y}" reflect_z="${reflect_z}" reflect_rotation="${True}" />
           </xacro:unless>
           <!-- Preserve the mesh's embedded materials. -->
@@ -44,8 +44,8 @@
           <xacro:property name="collision_cfg" value="${collision_override if collision_override != 'none' else collisions[source_name]}" lazy_eval="false" />
           <xacro:if value="${frame_shift != 'none'}">
-            <xacro:openarm_emit_composed_origin first="${frame_shift}" second="${collision_cfg.origin}" reflect_x="${reflect_x}" reflect_y="${reflect_y}" reflect_z="${reflect_z}" />
+            <xacro:openarm_emit_shifted_origin frame_shift="${frame_shift}" origin="${collision_cfg.origin}" reflect_x="${reflect_x}" reflect_y="${reflect_y}" reflect_z="${reflect_z}" reflect_rotation="${True}" />
           </xacro:if>
           <xacro:unless value="${frame_shift != 'none'}">
-            <xacro:openarm_emit_origin origin="${collision_cfg.origin}" reflect_x="${reflect_x}" reflect_y="${reflect_y}" reflect_z="${reflect_z}" />
+            <xacro:openarm_emit_origin origin="${collision_cfg.origin}" reflect_x="${reflect_x}" reflect_y="${reflect_y}" reflect_z="${reflect_z}" reflect_rotation="${True}" />
           </xacro:unless>
           <geometry>
@@ -61,8 +61,8 @@
         <inertial>
           <xacro:if value="${frame_shift != 'none'}">
-            <xacro:openarm_emit_composed_origin first="${frame_shift}" second="${inertial_cfg.origin}" reflect_x="${reflect_x}" reflect_y="${reflect_y}" reflect_z="${reflect_z}" />
+            <xacro:openarm_emit_shifted_origin frame_shift="${frame_shift}" origin="${inertial_cfg.origin}" reflect_x="${reflect_x}" reflect_y="${reflect_y}" reflect_z="${reflect_z}" reflect_rotation="${True}" />
           </xacro:if>
           <xacro:unless value="${frame_shift != 'none'}">
-            <xacro:openarm_emit_origin origin="${inertial_cfg.origin}" reflect_x="${reflect_x}" reflect_y="${reflect_y}" reflect_z="${reflect_z}" />
+            <xacro:openarm_emit_origin origin="${inertial_cfg.origin}" reflect_x="${reflect_x}" reflect_y="${reflect_y}" reflect_z="${reflect_z}" reflect_rotation="${True}" />
           </xacro:unless>
           <mass value="${inertial_cfg.mass}" />
@@ -83,5 +83,5 @@
     <joint name="${joint_name}" type="${joint_type}">
       <xacro:if value="${frame_shift != 'none'}">
-        <xacro:openarm_emit_composed_origin first="${frame_shift}" second="${joint_origin_cfg}" reflect_x="${reflect_x}" reflect_y="${reflect_y}" reflect_z="${reflect_z}" reflect_rotation="${reflect_rotation}" />
+        <xacro:openarm_emit_shifted_origin frame_shift="${frame_shift}" origin="${joint_origin_cfg}" reflect_x="${reflect_x}" reflect_y="${reflect_y}" reflect_z="${reflect_z}" reflect_rotation="${reflect_rotation}" />
       </xacro:if>
       <xacro:unless value="${frame_shift != 'none'}">

File: assets/component_loader.xacro (robot description, xacro)
@@ -151,4 +151,5 @@
         joint_limits="${component_desc['joint_limits']}"
         joint_mimics="${component_desc['joint_mimics']}"
+        origin_override_joints="${component_runtime['origin_override_joints']}"
         inertials="${component_desc['inertials']}"
         visuals="${component_desc['visuals']}"
@@ -186,4 +187,5 @@
         reflect_include_joints="${component_runtime['reflect_include_joints']}"
         reflect_include_reference_points="${component_runtime['reflect_include_reference_points']}"
+        origin_override_joints="${component_runtime['origin_override_joints']}"
         limit_override_joints="${component_runtime['limit_override_joints']}"
         emit_grasp_frame="${emit_grasp_frame}"

File: assets/end_effector/pinch_gripper/urdf/pinch_gripper_macro.xacro (robot description, xacro)
@@ -17,5 +17,5 @@
   <xacro:include filename="$(find openarm_description)/assets/common/validation.xacro" />
   <xacro:macro name="openarm_pinch_gripper"
-    params="prefix connected_to mount_origin:=none topology joint_origins joint_axes joint_limits joint_mimics inertials visuals collisions reflect_x:=1 reflect_y:=1 reflect_z:=1 component_reflects:=false reflect_include_links:=^ reflect_include_joints:=^ reflect_include_reference_points:=^ limit_override_joints:=^ ee_reference_points:=^ emit_grasp_frame:=false grasp_reference_point:=grasp_frame skip_mount_joint:=false base_frame_shift:=none">
+    params="prefix connected_to mount_origin:=none topology joint_origins joint_axes joint_limits joint_mimics inertials visuals collisions reflect_x:=1 reflect_y:=1 reflect_z:=1 component_reflects:=false reflect_include_links:=^ reflect_include_joints:=^ reflect_include_reference_points:=^ origin_override_joints:=${dict()} limit_override_joints:=^ ee_reference_points:=^ emit_grasp_frame:=false grasp_reference_point:=grasp_frame skip_mount_joint:=false base_frame_shift:=none">
     <xacro:property name="base_link_name" value="${topology['links'][0]}" />
     <xacro:property name="base_link_full_name" value="${prefix}${base_link_name}" />
@@ -41,60 +41,11 @@
     <xacro:property name="finger1_mimic_override" value="${dict(joint=finger1_mimic_target_name, multiplier=joint_mimics[finger1_joint_source]['multiplier'], offset=joint_mimics[finger1_joint_source]['offset']) if finger1_has_mimic else 'none'}" />
     <xacro:property name="finger2_mimic_override" value="${dict(joint=finger2_mimic_target_name, multiplier=joint_mimics[finger2_joint_source]['multiplier'], offset=joint_mimics[finger2_joint_source]['offset']) if finger2_has_mimic else 'none'}" />
-    <!-- The base link is emitted inline because its naming and frame-shift behavior differ from the finger links. -->
-    <link name="${base_link_full_name}">
-      <xacro:if value="${base_link_name in visuals}">
-        <visual name="${base_link_full_name}_visual">
-          <xacro:property name="base_visual_cfg" value="${visuals[base_link_name]}" lazy_eval="false" />
-          <xacro:if value="${use_base_frame_shift}">
-            <xacro:openarm_emit_composed_origin first="${resolved_base_frame_shift}" second="${base_visual_cfg.origin}" reflect_x="${reflect_x if base_link_reflects else 1}" reflect_y="${reflect_y if base_link_reflects else 1}" reflect_z="${reflect_z if base_link_reflects else 1}" />
-          </xacro:if>
-          <xacro:unless value="${use_base_frame_shift}">
-            <xacro:openarm_emit_origin origin="${base_visual_cfg.origin}" reflect_x="${reflect_x if base_link_reflects else 1}" reflect_y="${reflect_y if base_link_reflects else 1}" reflect_z="${reflect_z if base_link_reflects else 1}" />
-          </xacro:unless>
-          <!-- Preserve the mesh's embedded materials. -->
-          <geometry>
-            <mesh
-              filename="${base_visual_cfg.geometry.mesh}"
-              scale="${(reflect_x if base_link_reflects else 1) * base_visual_cfg.geometry.scale.x} ${(reflect_y if base_link_reflects else 1) * base_visual_cfg.geometry.scale.y} ${(reflect_z if base_link_reflects else 1) * base_visual_cfg.geometry.scale.z}" />
-          </geometry>
-        </visual>
-      </xacro:if>
-      <xacro:if value="${base_link_name in collisions}">
-        <collision name="${base_link_full_name}_collision">
-          <xacro:property name="base_collision_cfg" value="${collisions[base_link_name]}" lazy_eval="false" />
-          <xacro:if value="${use_base_frame_shift}">
-            <xacro:openarm_emit_composed_origin first="${resolved_base_frame_shift}" second="${base_collision_cfg.origin}" reflect_x="${reflect_x if base_link_reflects else 1}" reflect_y="${reflect_y if base_link_reflects else 1}" reflect_z="${reflect_z if base_link_reflects else 1}" />
-          </xacro:if>
-          <xacro:unless value="${use_base_frame_shift}">
-            <xacro:openarm_emit_origin origin="${base_collision_cfg.origin}" reflect_x="${reflect_x if base_link_reflects else 1}" reflect_y="${reflect_y if base_link_reflects else 1}" reflect_z="${reflect_z if base_link_reflects else 1}" />
-          </xacro:unless>
-          <geometry>
-            <mesh
-              filename="${base_collision_cfg.geometry.mesh}"
-              scale="${(reflect_x if base_link_reflects else 1) * base_collision_cfg.geometry.scale.x} ${(reflect_y if base_link_reflects else 1) * base_collision_cfg.geometry.scale.y} ${(reflect_z if base_link_reflects else 1) * base_collision_cfg.geometry.scale.z}" />
-          </geometry>
-        </collision>
-      </xacro:if>
-      <xacro:if value="${base_link_name in inertials}">
-        <xacro:property name="base_inertial_cfg" value="${inertials[base_link_name]}" lazy_eval="false" />
-        <xacro:property name="base_inertia_terms" value="${base_inertial_cfg.inertia}" lazy_eval="false" />
-        <inertial>
-          <xacro:if value="${use_base_frame_shift}">
-            <xacro:openarm_emit_composed_origin first="${resolved_base_frame_shift}" second="${base_inertial_cfg.origin}" reflect_x="${reflect_x if base_link_reflects else 1}" reflect_y="${reflect_y if base_link_reflects else 1}" reflect_z="${reflect_z if base_link_reflects else 1}" />
-          </xacro:if>
-          <xacro:unless value="${use_base_frame_shift}">
-            <xacro:openarm_emit_origin origin="${base_inertial_cfg.origin}" reflect_x="${reflect_x if base_link_reflects else 1}" reflect_y="${reflect_y if base_link_reflects else 1}" reflect_z="${reflect_z if base_link_reflects else 1}" />
-          </xacro:unless>
-          <mass value="${base_inertial_cfg.mass}" />
-          <inertia
-            ixx="${base_inertia_terms.xx}"
-            ixy="${(reflect_x if base_link_reflects else 1) * (reflect_y if base_link_reflects else 1) * base_inertia_terms.xy}"
-            ixz="${(reflect_x if base_link_reflects else 1) * (reflect_z if base_link_reflects else 1) * base_inertia_terms.xz}"
-            iyy="${base_inertia_terms.yy}"
-            iyz="${(reflect_y if base_link_reflects else 1) * (reflect_z if base_link_reflects else 1) * base_inertia_terms.yz}"
-            izz="${base_inertia_terms.zz}" />
-        </inertial>
-      </xacro:if>
-    </link>
+    <xacro:openarm_emit_link
+      link_name="${base_link_full_name}" source_name="${base_link_name}"
+      inertials="${inertials}" visuals="${visuals}" collisions="${collisions}"
+      reflect_x="${reflect_x if base_link_reflects else 1}"
+      reflect_y="${reflect_y if base_link_reflects else 1}"
+      reflect_z="${reflect_z if base_link_reflects else 1}"
+      frame_shift="${base_frame_shift}" />
     <xacro:openarm_emit_link
       link_name="${prefix}${finger1_source}"
@@ -116,5 +67,5 @@
       reflect_z="${reflect_z if finger2_link_reflects else 1}" />
     <xacro:unless value="${skip_mount_joint}">
-      <joint name="${prefix}ee_mount_joint" type="fixed">
+      <joint name="${base_link_full_name}_mount_joint" type="fixed">
         <xacro:openarm_emit_origin origin="${resolved_mount_origin}" />
         <parent link="${connected_to}" />
@@ -123,15 +74,15 @@
     </xacro:unless>
     <!-- Finger joints are emitted explicitly so mimic remapping stays local to the EE emitter. -->
-    <xacro:property name="finger1_joint_origin_cfg" value="${joint_origins[finger1_joint_source]['origin']}" lazy_eval="false" />
-    <xacro:property name="finger2_joint_origin_cfg" value="${joint_origins[finger2_joint_source]['origin']}" lazy_eval="false" />
+    <xacro:property name="finger1_joint_origin_cfg" value="${origin_override_joints.get(finger1_joint_source, joint_origins[finger1_joint_source]['origin'])}" lazy_eval="false" />
+    <xacro:property name="finger2_joint_origin_cfg" value="${origin_override_joints.get(finger2_joint_source, joint_origins[finger2_joint_source]['origin'])}" lazy_eval="false" />
     <xacro:property name="finger1_joint_axis_cfg" value="${joint_axes[finger1_joint_source]['axis']}" lazy_eval="false" />
     <xacro:property name="finger2_joint_axis_cfg" value="${joint_axes[finger2_joint_source]['axis']}" lazy_eval="false" />
     <xacro:property
       name="finger1_joint_axis_reflect_sign"
-      value="${-1 if ((reflect_x == -1 and finger1_joint_axis_cfg.x * finger1_joint_axis_cfg.x > 1e-18) or (reflect_y == -1 and finger1_joint_axis_cfg.y * finger1_joint_axis_cfg.y > 1e-18) or (reflect_z == -1 and finger1_joint_axis_cfg.z * finger1_joint_axis_cfg.z > 1e-18)) else 1}"
+      value="${-1 if finger1_joint_reflects and ((reflect_x == -1 and finger1_joint_axis_cfg.x * finger1_joint_axis_cfg.x > 1e-18) or (reflect_y == -1 and finger1_joint_axis_cfg.y * finger1_joint_axis_cfg.y > 1e-18) or (reflect_z == -1 and finger1_joint_axis_cfg.z * finger1_joint_axis_cfg.z > 1e-18)) else 1}"
       lazy_eval="false" />
     <xacro:property
       name="finger2_joint_axis_reflect_sign"
-      value="${-1 if ((reflect_x == -1 and finger2_joint_axis_cfg.x * finger2_joint_axis_cfg.x > 1e-18) or (reflect_y == -1 and finger2_joint_axis_cfg.y * finger2_joint_axis_cfg.y > 1e-18) or (reflect_z == -1 and finger2_joint_axis_cfg.z * finger2_joint_axis_cfg.z > 1e-18)) else 1}"
+      value="${-1 if finger2_joint_reflects and ((reflect_x == -1 and finger2_joint_axis_cfg.x * finger2_joint_axis_cfg.x > 1e-18) or (reflect_y == -1 and finger2_joint_axis_cfg.y * finger2_joint_axis_cfg.y > 1e-18) or (reflect_z == -1 and finger2_joint_axis_cfg.z * finger2_joint_axis_cfg.z > 1e-18)) else 1}"
       lazy_eval="false" />
     <xacro:property name="finger1_joint_limit_cfg" value="${joint_limits[finger1_joint_source]['limit']}" lazy_eval="false" />
@@ -165,8 +116,8 @@
     <joint name="${prefix}${finger1_joint_source}" type="${topology['joints'][finger1_joint_source]['type']}">
       <xacro:if value="${use_base_frame_shift}">
-        <xacro:openarm_emit_composed_origin first="${resolved_base_frame_shift}" second="${finger1_joint_origin_cfg}" reflect_x="${reflect_x if finger1_joint_reflects else 1}" reflect_y="${reflect_y if finger1_joint_reflects else 1}" reflect_z="${reflect_z if finger1_joint_reflects else 1}" />
+        <xacro:openarm_emit_shifted_origin frame_shift="${resolved_base_frame_shift}" origin="${finger1_joint_origin_cfg}" reflect_x="${reflect_x if finger1_joint_reflects else 1}" reflect_y="${reflect_y if finger1_joint_reflects else 1}" reflect_z="${reflect_z if finger1_joint_reflects else 1}" reflect_rotation="${True}" />
       </xacro:if>
       <xacro:unless value="${use_base_frame_shift}">
-        <xacro:openarm_emit_origin origin="${finger1_joint_origin_cfg}" reflect_x="${reflect_x if finger1_joint_reflects else 1}" reflect_y="${reflect_y if finger1_joint_reflects else 1}" reflect_z="${reflect_z if finger1_joint_reflects else 1}" />
+        <xacro:openarm_emit_origin origin="${finger1_joint_origin_cfg}" reflect_x="${reflect_x if finger1_joint_reflects else 1}" reflect_y="${reflect_y if finger1_joint_reflects else 1}" reflect_z="${reflect_z if finger1_joint_reflects else 1}" reflect_rotation="${True}" />
       </xacro:unless>
       <parent link="${prefix}${topology['joints'][finger1_joint_source]['parent']}" />
@@ -185,8 +136,8 @@
     <joint name="${prefix}${finger2_joint_source}" type="${topology['joints'][finger2_joint_source]['type']}">
       <xacro:if value="${use_base_frame_shift}">
-        <xacro:openarm_emit_composed_origin first="${resolved_base_frame_shift}" second="${finger2_joint_origin_cfg}" reflect_x="${reflect_x if finger2_joint_reflects else 1}" reflect_y="${reflect_y if finger2_joint_reflects else 1}" reflect_z="${reflect_z if finger2_joint_reflects else 1}" />
+        <xacro:openarm_emit_shifted_origin frame_shift="${resolved_base_frame_shift}" origin="${finger2_joint_origin_cfg}" reflect_x="${reflect_x if finger2_joint_reflects else 1}" reflect_y="${reflect_y if finger2_joint_reflects else 1}" reflect_z="${reflect_z if finger2_joint_reflects else 1}" reflect_rotation="${True}" />
       </xacro:if>
       <xacro:unless value="${use_base_frame_shift}">
-        <xacro:openarm_emit_origin origin="${finger2_joint_origin_cfg}" reflect_x="${reflect_x if finger2_joint_reflects else 1}" reflect_y="${reflect_y if finger2_joint_reflects else 1}" reflect_z="${reflect_z if finger2_joint_reflects else 1}" />
+        <xacro:openarm_emit_origin origin="${finger2_joint_origin_cfg}" reflect_x="${reflect_x if finger2_joint_reflects else 1}" reflect_y="${reflect_y if finger2_joint_reflects else 1}" reflect_z="${reflect_z if finger2_joint_reflects else 1}" reflect_rotation="${True}" />
       </xacro:unless>
       <parent link="${prefix}${topology['joints'][finger2_joint_source]['parent']}" />
