Commit message: Configure empty arm-tip folding in topology

File: assets/common/assembly.xacro (robot description, xacro)
@@ -29,5 +29,5 @@
   </xacro:macro>
   <xacro:macro name="openarm_resolve_component_runtime"
-    params="component_api component_name components robot_preset config_root root_frame component_cfg component_desc parent_desc:=none collapse_internal_empty_links:=false emit_grasp_frame:=false out_name">
+    params="component_api component_name components robot_preset config_root root_frame component_cfg component_desc parent_desc:=none emit_grasp_frame:=false out_name">
     <xacro:property name="none_value" value="${'none'}" lazy_eval="false" />
     <xacro:property name="zero_origin" value="${dict(x=0.0, y=0.0, z=0.0, roll=0.0, pitch=0.0, yaw=0.0)}" lazy_eval="false" />
@@ -127,5 +127,5 @@
       lazy_eval="false" />
     <xacro:openarm_collect_collapsible_children names="${collapse_candidate_names}" robot_preset="${robot_preset}"
-      component_api="${component_api}" options="${dict(emit_grasp_frame=emit_grasp_frame, collapse_empty_end=collapse_internal_empty_links)}" out_name="candidate_descriptions" />
+      component_api="${component_api}" options="${dict(emit_grasp_frame=emit_grasp_frame)}" out_name="candidate_descriptions" />
     <xacro:openarm_require condition="${len(candidate_descriptions) &lt;= 1}"
       message="${'Invalid robot preset: component %s has multiple children competing to collapse the same terminal empty link.' % component_name}" />
@@ -160,5 +160,5 @@
   </xacro:macro>
   <xacro:macro name="openarm_emit_component_tree"
-    params="component_api component_name components robot_preset config_root root_frame parent_desc:=none preloaded_desc:=none collapse_internal_empty_links:=false emit_grasp_frame:=false">
+    params="component_api component_name components robot_preset config_root root_frame parent_desc:=none preloaded_desc:=none emit_grasp_frame:=false">
     <xacro:property name="none_value" value="${'none'}" lazy_eval="false" />
     <xacro:property name="component_cfg" value="${robot_preset[component_name]}" lazy_eval="false" />
@@ -168,5 +168,5 @@
         component_name="${component_name}"
         component_cfg="${component_cfg}"
-        out_name="component_desc" options="${dict(emit_grasp_frame=emit_grasp_frame, collapse_empty_end=collapse_internal_empty_links)}" />
+        out_name="component_desc" options="${dict(emit_grasp_frame=emit_grasp_frame)}" />
     </xacro:if>
     <xacro:openarm_resolve_component_runtime component_api="${component_api}"
@@ -179,5 +179,4 @@
       component_desc="${component_desc}"
       parent_desc="${parent_desc}"
-      collapse_internal_empty_links="${collapse_internal_empty_links}"
       emit_grasp_frame="${emit_grasp_frame}"
       out_name="component_runtime" />
@@ -188,5 +187,5 @@
       component_desc="${component_desc}"
       component_runtime="${component_runtime}"
-      options="${dict(emit_grasp_frame=emit_grasp_frame, collapse_empty_end=collapse_internal_empty_links)}" />
+      options="${dict(emit_grasp_frame=emit_grasp_frame)}" />
     <xacro:openarm_emit_attached_components component_api="${component_api}"
       index="0"
@@ -199,9 +198,8 @@
       preloaded_component_name="${component_runtime['collapse_child_name']}"
       preloaded_component_desc="${component_runtime['collapse_child_desc']}"
-      collapse_internal_empty_links="${collapse_internal_empty_links}"
       emit_grasp_frame="${emit_grasp_frame}" />
   </xacro:macro>
   <xacro:macro name="openarm_emit_attached_components"
-    params="component_api index components parent_component_name robot_preset config_root root_frame parent_desc:=none preloaded_component_name:=none preloaded_component_desc:=none collapse_internal_empty_links:=false emit_grasp_frame:=false">
+    params="component_api index components parent_component_name robot_preset config_root root_frame parent_desc:=none preloaded_component_name:=none preloaded_component_desc:=none emit_grasp_frame:=false">
     <xacro:if value="${index &lt; len(components)}">
       <xacro:property name="none_value" value="${'none'}" lazy_eval="false" />
@@ -224,5 +222,4 @@
           parent_desc="${none_value if is_root_component else parent_desc}"
           preloaded_desc="${component_desc_override}"
-          collapse_internal_empty_links="${collapse_internal_empty_links}"
           emit_grasp_frame="${emit_grasp_frame}" />
       </xacro:if>
@@ -237,10 +234,9 @@
         preloaded_component_name="${preloaded_component_name}"
         preloaded_component_desc="${preloaded_component_desc}"
-        collapse_internal_empty_links="${collapse_internal_empty_links}"
         emit_grasp_frame="${emit_grasp_frame}" />
     </xacro:if>
   </xacro:macro>
   <xacro:macro name="openarm_assemble_robot"
-    params="component_api config_root robot_preset collapse_internal_empty_links:=false emit_grasp_frame:=false">
+    params="component_api config_root robot_preset emit_grasp_frame:=false">
     <xacro:property name="robot_cfg" value="${robot_preset['robot']}" lazy_eval="false" />
     <xacro:property name="root_frame" value="${robot_cfg['root_frame']}" lazy_eval="false" />
@@ -257,5 +253,4 @@
       config_root="${config_root}"
       root_frame="${root_frame}"
-      collapse_internal_empty_links="${collapse_internal_empty_links}"
       emit_grasp_frame="${emit_grasp_frame}" />
   </xacro:macro>

File: assets/common/components.xacro (robot description, xacro)
@@ -44,5 +44,5 @@
     <xacro:property name="component_root_link_actual" value="${component_cfg['link_name'] if component_type == 'body' else (component_prefix + component_topology['links'][0])}" lazy_eval="false" />
     <xacro:property name="component_default_mount_parent" value="${component_cfg['link_name'] if component_type == 'body' else (component_prefix + component_topology['links'][-1])}" lazy_eval="false" />
-    <xacro:property name="component_collapse_empty_end" value="${component_type == 'arm' and options.get('collapse_empty_end', False) and len([j for j in component_topology['joints'] if component_topology['joints'][j]['parent'] == component_topology['links'][-1]]) == 0}" lazy_eval="false" />
+    <xacro:property name="component_collapse_empty_end" value="${component_topology.get('collapse_empty_end', False) and len([j for j in component_topology['joints'] if component_topology['joints'][j]['parent'] == component_topology['links'][-1]]) == 0}" lazy_eval="false" />
     <xacro:property
       name="${out_name}"

File: assets/robot/openarm_v2.0/urdf/openarm_v20.urdf.xacro (robot description, xacro)
@@ -16,5 +16,4 @@
   <xacro:include filename="$(find openarm_description)/assets/robot/openarm_v2.0/urdf/ros2_control/openarm.bimanual.ros2_control.xacro" />
   <xacro:arg name="robot_preset" default="default_bimanual" />
-  <xacro:arg name="collapse_internal_empty_links" default="true" />
   <xacro:arg name="emit_grasp_frame" default="false" />
   <xacro:arg name="use_fake_hardware" default="true" />
@@ -28,5 +27,4 @@
     config_root="${config_root}"
     robot_preset="${robot_preset_cfg}"
-    collapse_internal_empty_links="$(arg collapse_internal_empty_links)"
     emit_grasp_frame="$(arg emit_grasp_frame)" />
   <xacro:property name="gains_file" value="${config_root}/arm/control/control_gains.yaml" />
