Commit message: Add accessory support and the default ZED Mini assembly

File: assets/robot/openarm_v2.0/urdf/example/v2.urdf (robot description, URDF)
Before this commit: robot openarm_v20, 24 links, 23 joints
Links:
- added link openarm_body_zed_camera_center; collision mesh filename=package://zed_description/meshes/zedm.stl; visual mesh filename=package://zed_description/meshes/zedm.stl
- added link openarm_body_zed_camera_link
- added link openarm_body_zed_left_camera_frame
- added link openarm_body_zed_left_camera_frame_optical
- added link openarm_body_zed_mount_base_link, mass 0.13704; visual mesh filename=package://openarm_description/assets/accessory/zed_mount/me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 scale=1 1 1
- added link openarm_body_zed_mount_camera_mount_point
- added link openarm_body_zed_right_camera_frame
- added link openarm_body_zed_right_camera_frame_optical
- added link openarm_camera_mount_point
Joints:
- added joint openarm_body_zed_camera_center_joint: type fixed, parent openarm_body_zed_camera_link, child openarm_body_zed_camera_center, origin xyz=0 0 0.01325 rpy=0 0.0 0
- added joint openarm_body_zed_left_camera_joint: type fixed, parent openarm_body_zed_camera_center, child openarm_body_zed_left_camera_frame, origin xyz=0.0 0.0315 0 rpy=0 0 0
- added joint openarm_body_zed_left_camera_optical_joint: type fixed, parent openarm_body_zed_left_camera_frame, child openarm_body_zed_left_camera_frame_optical, origin xyz=0 0 0 rpy=-1.5707963267948966 0.0 -1.5707963267948966
- added joint openarm_body_zed_mount_base_link_mount_joint: type fixed, parent openarm_camera_mount_point, child openarm_body_zed_mount_base_link, origin xyz=0.0 0.0 0.0 rpy=0.0 0.0 0.0
- added joint openarm_body_zed_mount_camera_mount_point_joint: type fixed, parent openarm_body_zed_mount_base_link, child openarm_body_zed_mount_camera_mount_point, origin xyz=0.0263085336684006 0.00869000000000031 0.065829226007701 rpy=0 1.08210413623648 0
- added joint openarm_body_zed_mount_joint: type fixed, parent openarm_body_zed_mount_camera_mount_point, child openarm_body_zed_camera_link, origin xyz=0.00119247 -0.007723415 8.746e-05 rpy=0.0 0.0 0.0
- added joint openarm_body_zed_right_camera_joint: type fixed, parent openarm_body_zed_camera_center, child openarm_body_zed_right_camera_frame, origin xyz=0.0 -0.0315 0 rpy=0 0 0
- added joint openarm_body_zed_right_camera_optical_joint: type fixed, parent openarm_body_zed_right_camera_frame, child openarm_body_zed_right_camera_frame_optical, origin xyz=0 0 0 rpy=-1.5707963267948966 0.0 -1.5707963267948966
- added joint openarm_camera_mount_point_joint: type fixed, parent openarm_body_link0, child openarm_camera_mount_point, origin xyz=0.03 0.0 0.743 rpy=0.0 0.0 0.0
