Commit message: Migrate V1 directly to shared presets and external bodies

File: assets/robot/openarm_v1.0/urdf/example/v1.urdf (robot description, URDF)
Before this commit: robot openarm, 26 links, 25 joints
Links:
- link openarm_body_link0: geometry collision mesh filename=package://openarm_description/assets/body/v1.0/meshes/colli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 scale=0.001 0.001 0.001; visual mesh filename=package://openarm_description/assets/body/v1.0/meshes/visua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 scale=0.001 0.001 0.001
- link openarm_left_link7: geometry collision mesh filename=package://openarm_description/assets/end_effector/parallel_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 scale=0.001 -0.001 0.001; visual mesh filename=package://openarm_description/assets/end_effector/parallel_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 scale=0.001 -0.001 0.001
- link openarm_right_link7: geometry collision mesh filename=package://openarm_description/assets/end_effector/parallel_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 scale=0.001 0.001 0.001; visual mesh filename=package://openarm_description/assets/end_effector/parallel_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 scale=0.001 0.001 0.001
Joints:
- removed joint openarm_body_world_joint
- removed joint openarm_left_openarm_body_link0_joint
- removed joint openarm_right_openarm_body_link0_joint
- added joint openarm_body_link0_mount_joint: type fixed, parent world, child openarm_body_link0, origin xyz=0.0 0.0 0.0 rpy=0.0 0.0 0.0
- added joint openarm_left_link0_mount_joint: type fixed, parent openarm_body_link0, child openarm_left_link0, origin xyz=0.0 0.03 0.697 rpy=-1.5708 -0.0 0.0
- added joint openarm_right_link0_mount_joint: type fixed, parent openarm_body_link0, child openarm_right_link0, origin xyz=0.0 -0.03 0.697 rpy=1.5708 -0.0 0.0
- joint openarm_left_finger_joint1: origin xyz=0.0 -0.005 0.015 rpy=0 0 0 -> xyz=0 -0.005 0.015 rpy=0 0 0
- joint openarm_left_finger_joint2: origin xyz=0.0 0.005 0.015 rpy=0 0 0 -> xyz=0 0.005 0.015 rpy=0 0 0
- joint openarm_left_hand_joint: origin xyz=0.0 0.0 0.1001 rpy=0 0 0 -> xyz=0.0 0.0 0.1001 rpy=0.0 -0.0 0.0
- joint openarm_left_joint1: limit lower=-3.490659 upper=1.3962629999999998 effort=40 velocity=16.754666 -> lower=-3.490659 upper=1.396263 effort=40 velocity=16.754666; origin xyz=0.0 0.0 0.0625 rpy=0 0 0 -> xyz=0.0 -0.0 0.0625 rpy=0 0 0
- joint openarm_left_joint2: origin xyz=-0.0301 0.0 0.06 rpy=-1.57079632679 0 0 -> xyz=-0.0301 -0.0 0.06 rpy=-1.57079632679 0 0
- joint openarm_left_joint3: origin xyz=0.0301 0.0 0.06625 rpy=0 0 0 -> xyz=0.0301 -0.0 0.06625 rpy=0 0 0
- joint openarm_left_joint4: origin xyz=-0.0 0.0315 0.15375 rpy=0 0 0 -> xyz=0.0 0.0315 0.15375 rpy=0 0 0
- joint openarm_left_joint6: origin xyz=0.0375 0.0 0.1205 rpy=0 0 0 -> xyz=0.0375 -0.0 0.1205 rpy=0 0 0
- joint openarm_left_joint7: origin xyz=-0.0375 0.0 0.0 rpy=0 0 0 -> xyz=-0.0375 -0.0 0.0 rpy=0 0 0
- joint openarm_right_finger_joint1: origin xyz=0.0 -0.005 0.015 rpy=0 0 0 -> xyz=0 -0.005 0.015 rpy=0 0 0
- joint openarm_right_finger_joint2: origin xyz=0.0 0.005 0.015 rpy=0 0 0 -> xyz=0 0.005 0.015 rpy=0 0 0
- joint openarm_right_hand_joint: origin xyz=0.0 0.0 0.1001 rpy=0 0 0 -> xyz=0.0 0.0 0.1001 rpy=0.0 -0.0 0.0
- joint openarm_right_joint4: origin xyz=-0.0 0.0315 0.15375 rpy=0 0 0 -> xyz=0.0 0.0315 0.15375 rpy=0 0 0

Commit message: Center V1 joint origins while preserving motor coordinates

File: assets/robot/openarm_v1.0/urdf/example/v1.urdf (robot description, URDF)
Before this commit: robot openarm, 26 links, 25 joints
Joints:
- joint openarm_left_joint2: origin xyz=-0.0301 -0.0 0.06 rpy=-1.57079632679 0 0 -> xyz=0.0 -0.0 0.06 rpy=-1.57079632679 0 0
- joint openarm_left_joint3: origin xyz=0.0301 -0.0 0.06625 rpy=0 0 0 -> xyz=0.0 -0.0 0.06625 rpy=0 0 0
- joint openarm_left_joint4: origin xyz=0.0 0.0315 0.15375 rpy=0 0 0 -> xyz=0.0 0.0 0.15375 rpy=0 0 0
- joint openarm_left_joint5: origin xyz=0.0 -0.0315 0.0955 rpy=0 0 0 -> xyz=0.0 -0.0 0.0955 rpy=0 0 0
- joint openarm_left_joint6: origin xyz=0.0375 -0.0 0.1205 rpy=0 0 0 -> xyz=0.0 -0.0 0.1205 rpy=0 0 0
- joint openarm_left_joint7: origin xyz=-0.0375 -0.0 0.0 rpy=0 0 0 -> xyz=0.0 -0.0 0.0 rpy=0 0 0
- joint openarm_right_joint2: origin xyz=-0.0301 0.0 0.06 rpy=1.57079632679 0 0 -> xyz=0.0 0.0 0.06 rpy=1.57079632679 0 0
- joint openarm_right_joint3: origin xyz=0.0301 0.0 0.06625 rpy=0 0 0 -> xyz=0.0 0.0 0.06625 rpy=0 0 0
- joint openarm_right_joint4: origin xyz=0.0 0.0315 0.15375 rpy=0 0 0 -> xyz=0.0 0.0 0.15375 rpy=0 0 0
- joint openarm_right_joint5: origin xyz=0.0 -0.0315 0.0955 rpy=0 0 0 -> xyz=0.0 0.0 0.0955 rpy=0 0 0
- joint openarm_right_joint6: origin xyz=0.0375 0.0 0.1205 rpy=0 0 0 -> xyz=0.0 0.0 0.1205 rpy=0 0 0
- joint openarm_right_joint7: origin xyz=-0.0375 0.0 0.0 rpy=0 0 0 -> xyz=0.0 0.0 0.0 rpy=0 0 0
